File: STM32F030C8T6.kicad_sch (KiCad schematic)
At the start: 29 parts, among them SW1 SW_Push, SW2 SW_Push, U1 STM32F030C8T6, U2 AMS1117-3.3

Commit message: Add files via upload
Parts:
- removed R6: 100KΩ, Resistor_SMD:R_0402_1005Metric, symbol Device:R
- R2: value 100KΩ -> 10KΩ; LCSC C25741 -> C25744
- R3: value 1KΩ -> 10KΩ; LCSC C11702 -> C25744
- XTAL2: footprint Crystal:Crystal_SMD_5032-2Pin_5.0x3.2mm -> Crystal:Crystal_SMD_HC49-SD; LCSC C115962 -> C12674
Connections:
- net +3.3V: now also R3.2
- net BOOT0: now also C5.1, R2.1, SW2.2; no longer R3.2
- net GND: now also R2.2; no longer R2.1
- net NRST: now also R3.1
